File: lfo_stomp_v1/lfo_stomp_v1.kicad_sch (KiCad schematic)
At the start: 50 parts, among them J1 Conn_02x05_Odd_Even, J2 SYNC_IN, J3 LFO_INV, J4 LFO, Q1 BC547, Q2 2N3906, SW1 SW_Push, U1 LM7805_TO220, U2 ElectricDruid_STOMPLFO, U3 TL072, U4 L78L05_SOT89

Commit message: Geographic reannotate
Parts:
- renumbered C11 to C10, C9 to C100, C8 to C101, C7 to C11, C10 to C12, C3 to C2, C6 to C3, C1 to C4, C4 to C5, C13 to C6, C5 to C7, C12 to C8, C2 to C9, D4 to D100, D1 to D2, D2 to D3, D3 to D4, FB2 to FB1, FB1 to FB2, J2 to J100, J4 to J101, J3 to J102, J1 to J2, LOGO1 to LOGO100, LOGO2 to LOGO101, LOGO3 to LOGO2, R8 to R10, R9 to R12, R10 to R13, R3 to R2, R2 to R3, R13 to R5, R7 to R6, R5 to R7, R6 to R8, R12 to R9, R_DEPTH1 to R_DEPTH100, R_FREQ1 to R_FREQ100, R_OFFSET1 to R_OFFSET100, R_WAVEFORM1 to R_WAVEFORM100, SW1 to SW100, U4 to U2, U2 to U4

Commit message: Page titles and fixed pot orientations
Connections:
- net +5V: now also R_DEPTH100.3, R_FREQ100.3, R_OFFSET100.3, R_WAVEFORM100.3; no longer R_DEPTH100.1, R_FREQ100.1, R_OFFSET100.1, R_WAVEFORM100.1
- net GND: now also R_DEPTH100.1, R_FREQ100.1, R_OFFSET100.1, R_WAVEFORM100.1; no longer R_DEPTH100.3, R_FREQ100.3, R_OFFSET100.3, R_WAVEFORM100.3
Other:
- company: (none) -> RobotDialogs
- title: (none) -> STOMPLFO 
Changed lines of the file:
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@@
 (kicad_sch (version 20211123) (generator eeschema)
   (paper "A4")
+  (title_block
+    (title "STOMPLFO ")
+    (date "2022-06-25")
+    (rev "1.0")
+    (company "RobotDialogs")
+  )
   (junction (at 76.835 35.56) (diameter 0) (color 0 0 0 0)
   )
@@
     (pin "1")
   )
-  (symbol (lib_id "Device:R_Potentiometer_MountingPin") (at 96.52 158.75 0) (unit 1)
-    (in_bom yes) (on_board yes)
-    (property "Reference" "R_FREQ100" (id 0) (at 90.17 154.94 0))
-    (property "Value" "B100K" (id 1) (at 90.17 162.56 0))
+  (symbol (lib_id "Device:R_Potentiometer_MountingPin") (at 96.52 158.75 0) (mirror x) (unit 1)
+    (in_bom yes) (on_board yes)
+    (property "Reference" "R_FREQ100" (id 0) (at 90.17 162.56 0))
+    (property "Value" "B100K" (id 1) (at 90.17 154.94 0))
     (property "Footprint" "My Stuff:Potentiometer_Alpha_RD901F-40-00D_Single_Vertical_w_3d" (id 2) (at 96.52 158.75 0)
       (effects (font (size 1.27 1.27)) hide)
@@
     (pin "2")
   )
-  (symbol (lib_id "Device:R_Potentiometer_MountingPin") (at 96.52 92.71 0) (unit 1)
-    (in_bom yes) (on_board yes)
-    (property "Reference" "R_OFFSET100" (id 0) (at 88.9 88.9 0))
-    (property "Value" "B100K" (id 1) (at 91.44 96.52 0))
+  (symbol (lib_id "Device:R_Potentiometer_MountingPin") (at 96.52 92.71 0) (mirror x) (unit 1)
+    (in_bom yes) (on_board yes)
+    (property "Reference" "R_OFFSET100" (id 0) (at 88.9 96.52 0))
+    (property "Value" "B100K" (id 1) (at 91.44 88.9 0))
     (property "Footprint" "My Stuff:Potentiometer_Alpha_RD901F-40-00D_Single_Vertical_w_3d" (id 2) (at 96.52 92.71 0)
       (effects (font (size 1.27 1.27)) hide)
@@
     (pin "1")
   )
-  (symbol (lib_id "Device:R_Potentiometer_MountingPin") (at 96.52 130.81 0) (unit 1)
-    (in_bom yes) (on_board yes)
-    (property "Reference" "R_DEPTH100" (id 0) (at 90.17 127 0))
-    (property "Value" "B100K" (id 1) (at 91.44 133.35 0))
+  (symbol (lib_id "Device:R_Potentiometer_MountingPin") (at 96.52 130.81 0) (mirror x) (unit 1)
+    (in_bom yes) (on_board yes)
+    (property "Reference" "R_DEPTH100" (id 0) (at 90.17 134.62 0))
+    (property "Value" "B100K" (id 1) (at 91.44 128.27 0))
     (property "Footprint" "My Stuff:Potentiometer_Alpha_RD901F-40-00D_Single_Vertical_w_3d" (id 2) (at 96.52 130.81 0)
       (effects (font (size 1.27 1.27)) hide)
@@
     (pin "MP")
   )
-  (symbol (lib_id "Device:R_Potentiometer_MountingPin") (at 96.52 144.78 0) (unit 1)
-    (in_bom yes) (on_board yes)
-    (property "Reference" "R_WAVEFORM100" (id 0) (at 86.36 140.97 0))
-    (property "Value" "B100K" (id 1) (at 90.17 148.59 0))
+  (symbol (lib_id "Device:R_Potentiometer_MountingPin") (at 96.52 144.78 0) (mirror x) (unit 1)
+    (in_bom yes) (on_board yes)
+    (property "Reference" "R_WAVEFORM100" (id 0) (at 86.36 148.59 0))
+    (property "Value" "B100K" (id 1) (at 90.17 140.97 0))
     (property "Footprint" "My Stuff:Potentiometer_Alpha_RD901F-40-00D_Single_Vertical_w_3d" (id 2) (at 96.52 144.78 0)
       (effects (font (size 1.27 1.27)) hide)

Commit message: Cleanup
Parts:
- removed Q2: 2N3906, Package_TO_SOT_THT:TO-92_Inline_Wide, symbol Transistor_BJT:2N3906
- added Q2: BC547, Package_TO_SOT_THT:TO-92_Inline_Wide, symbol Transistor_BJT:BC547
- D100: value LED? -> LED
- R1: value 100k -> 10k
- R10: value 100k -> 2k
- R11: value 22k -> 10k
- R9: value 3.3k -> 10k
Connections:
- net +12V: now also D100.2 (A); no longer R9.1
- net GND: now also Q2.3 (E); no longer D100.1 (K)
- net at R13.1, R6.2, U3.1: no longer R10.2
- net at R3.1, U4.3 (PDM_OUT): now also R10.2
- net at R9.2: now also Q2.1 (C); no longer D100.2 (A)
- net at R10.1, R11.1: now also Q2.2 (B)
- new net: D100.1 (K), R9.1
Other:
- moved on the sheet: C11, D100, R10, R11, R9
